File: Modules/Jack Converter/Panel.kicad_sch (KiCad schematic)
At the start: 0 parts

Commit message: Deleted Panel sch sheet
Parts:
- added H2, H3, H4, H5: MountingHole_Pad, SynthStuff:MountingHole_3.2mm_M3_Pad4mm, symbol Mechanical:MountingHole_Pad
Connections:
- new net GND: H2.1, H3.1, H4.1, H5.1
